Commit message: lower leg

File: riser_robot_description/urdf/leg.xacro (robot description, xacro)
@@ -39,4 +39,20 @@
 	  </visual>
   </link>
+  <link name="${name}_lower_leg_link">
+		<pose>0 0 0 0 0 0</pose>
+		<xacro:cylinder_inertial mass="${holder_weight}" radius="${holder_radius}" length="${holder_length}"/>
+		<collision>
+			<origin rpy="0 0 0" xyz="0 0 0"/>
+			<geometry>
+		  	<cylinder length="${holder_length}" radius="${holder_radius}"/>
+			</geometry>
+		</collision>
+		<visual>
+			<origin rpy="0 0 0" xyz="0 0 0"/>
+		  <geometry>
+		  	<cylinder length="${holder_length}" radius="${holder_radius}"/>
+		  </geometry>
+	  </visual>
+  </link>
 	<!-- JOINTS -->
 	<joint name="${name}_leg_joint" type="fixed">
@@ -50,4 +66,9 @@
 			<origin xyz="0 -${holder_radius/2 + pipe_length/2} 0" rpy="-${pi/2} 0 0"/>
 	</joint>
+	<joint name="${name}_lower_leg_joint" type="fixed">
+			<child link="${name}_lower_leg_link"/>
+			<parent link="${name}_upper_pipe"/>
+			<origin xyz="0 -${holder_radius/2 + pipe_length/2} 0" rpy="-${pi/2} 0 0"/>
+	</joint>
 	</xacro:macro>
 </robot>

File: riser_robot_description/urdf/riser_robot.xacro (robot description, xacro)
@@ -22,5 +22,5 @@
   <xacro:property name="holder_length" value="${chassis_height/2 + 0.05}" />
   <xacro:property name="pipe_radius" value="0.05" />
-  <xacro:property name="pipe_length" value="0.3" />
+  <xacro:property name="pipe_length" value="0.4" />
   <gazebo reference="base_link">
     <material>Gazebo/Orange</material>
